File: kicad/AMP_ma12070_HQ.kicad_sch (KiCad schematic)
At the start: 21 parts

Commit message: minor changes
Other:
- note added: "ANALOG BLT Config: * MSEL0 > 5V * MSEL1 > GND * AC-coupling Caps are used (see Table 9-2 page 23)"
- note added: "DIGITAL BLT Config: * SD1 > GND * SCLK and WS must be in sync with CLK * MSELO > 5V * MSEL1 > GND"
- note added: "MUTE / ENABLE: * /MUTE: MUTE audio when pulled LOW * /ENABLE: keep device in inactive state while pulled HIGH"
- note removed: "SCLK and WS must be syncronised with CLK"
- note removed: "SE/BTL/PBTL configuration"
- note removed: "pull high for inactive state"
Changed lines of the file:
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@@
     (stroke (width 0) (type default) (color 0 0 0 0))
-  )
-  (text "SCLK and WS must be syncronised with CLK" (at 121.92 27.94 0)
-    (effects (font (size 1 1)) (justify left bottom))
   )
   (text "ANALOG / DIGITAL INPUT" (at 29.21 99.06 0)
     (effects (font (size 1.27 1.27)) (justify left bottom))
   )
-  (text "pull high for inactive state" (at 123.19 74.93 0)
+  (text "ANALOG BLT Config:\n* MSEL0 > 5V\n* MSEL1 > GND \n* AC-coupling Caps are used (see Table 9-2 page 23)"
+    (at 96.52 50.8 0)
+    (effects (font (size 1 1)) (justify left bottom))
+  )
+  (text "MUTE / ENABLE:\n* /MUTE: MUTE audio when pulled LOW\n* /ENABLE: keep device in inactive state while pulled HIGH\n"
+    (at 97.79 74.93 0)
     (effects (font (size 1 1)) (justify left bottom))
   )
@@
     (effects (font (size 1.27 1.27)) (justify left bottom))
   )
+  (text "DIGITAL BLT Config:\n* SD1 > GND \n* SCLK and WS must be in sync with CLK \n* MSELO > 5V \n* MSEL1 > GND"
+    (at 96.52 33.02 0)
+    (effects (font (size 1 1)) (justify left bottom))
+  )
   (text "I2C Control\n\n" (at 27.94 153.67 0)
     (effects (font (size 1.27 1.27)) (justify left bottom))
   )
-  (text "SE/BTL/PBTL configuration " (at 124.46 59.69 0)
-    (effects (font (size 1 1)) (justify left bottom))
-  )
   (label "MSEL0" (at 204.47 128.27 180)
